Commit message: wl4v2 can walk to stair in 3200 ot

File: resources/wl4/urdf/robot.urdf (robot description, URDF)
Before this commit: robot wl4_description, 19 links, 18 joints
Links:
- removed link base
- removed link imu_link
- added link imu, mass 0.001; collision box size=.001 .001 .001; visual box size=0.001 0.001 0.001
- link FL_calf: mass 2.053 -> 1.13
- link FL_foot: mass 0.918 -> 0.6; geometry collision cylinder length=0.0415 radius=0.0875; visual cylinder length=0.0415 radius=0.0875
- link FL_hip: mass 2.256 -> 1.7
- link FL_thigh: mass 3.591 -> 3.04
- link FR_calf: mass 2.053 -> 1.13
- link FR_foot: mass 0.918 -> 0.6; geometry collision cylinder length=0.0415 radius=0.0875; visual cylinder length=0.0415 radius=0.0875
- link FR_hip: mass 2.256 -> 1.7
- link FR_thigh: mass 3.591 -> 3.04
- link RL_calf: mass 2.053 -> 1.13
- link RL_foot: mass 0.918 -> 0.6; geometry collision cylinder length=0.0415 radius=0.0875; visual cylinder length=0.0415 radius=0.0875
- link RL_hip: mass 2.256 -> 1.7
- link RL_thigh: mass 3.591 -> 3.04
- link RR_calf: mass 2.053 -> 1.13
- link RR_foot: mass 0.918 -> 0.6; geometry collision cylinder length=0.0415 radius=0.0875; visual cylinder length=0.0415 radius=0.0875
- link RR_hip: mass 2.256 -> 1.7
- link RR_thigh: mass 3.591 -> 3.04
- link trunk: mass 35.606 -> 8.1
Joints:
- removed joint floating_base
- joint FL_calf_joint: limit lower=-2.7 upper=-0.4 effort=320 velocity=14 -> lower=-2.775 upper=-0.855 effort=60 velocity=20
- joint FL_foot_joint: limit lower=-1000000.0 upper=1000000.0 effort=320 velocity=14 -> lower=-1000000.0 upper=1000000.0 effort=20 velocity=25; origin xyz=0 0.05 -0.25 rpy=0 0 0 -> xyz=0 0.08295 -0.25 rpy=0 0 0
- joint FL_hip_joint: limit lower=-0.87 upper=0.87 effort=200 velocity=23 -> lower=-0.7853981633974483 upper=0.7853981633974483 effort=60 velocity=20; origin xyz=0.1875 0.075 0 rpy=0 0 0 -> xyz=0.1875 0.0725 0 rpy=0 0 0
- joint FL_thigh_joint: limit lower=-1.25 upper=1.25 effort=200 velocity=23 -> lower=-1.5707963267948966 upper=3.141592653589793 effort=60 velocity=20
- joint FR_calf_joint: limit lower=-2.7 upper=-0.4 effort=320 velocity=14 -> lower=-2.775 upper=-0.855 effort=60 velocity=20
- joint FR_foot_joint: limit lower=-1000000.0 upper=1000000.0 effort=320 velocity=14 -> lower=-1000000.0 upper=1000000.0 effort=20 velocity=25; origin xyz=0 -0.05 -0.25 rpy=0 0 0 -> xyz=0 -0.08295 -0.25 rpy=0 0 0
- joint FR_hip_joint: limit lower=-0.87 upper=0.87 effort=200 velocity=23 -> lower=-0.7853981633974483 upper=0.7853981633974483 effort=60 velocity=20; origin xyz=0.1875 -0.075 0 rpy=0 0 0 -> xyz=0.1875 -0.0725 0 rpy=0 0 0
- joint FR_thigh_joint: limit lower=-1.25 upper=1.25 effort=200 velocity=23 -> lower=-1.5707963267948966 upper=3.141592653589793 effort=60 velocity=20
- joint RL_calf_joint: limit lower=-2.7 upper=-0.4 effort=320 velocity=14 -> lower=-2.775 upper=-0.855 effort=60 velocity=20
- joint RL_foot_joint: limit lower=-1000000.0 upper=1000000.0 effort=320 velocity=14 -> lower=-1000000.0 upper=1000000.0 effort=20 velocity=25; origin xyz=0 0.05 -0.25 rpy=0 0 0 -> xyz=0 0.08295 -0.25 rpy=0 0 0
- joint RL_hip_joint: limit lower=-0.87 upper=0.87 effort=200 velocity=23 -> lower=-0.7853981633974483 upper=0.7853981633974483 effort=60 velocity=20; origin xyz=-0.1875 0.075 0 rpy=0 0 0 -> xyz=-0.1875 0.0725 0 rpy=0 0 0
- joint RL_thigh_joint: limit lower=-1.25 upper=1.25 effort=200 velocity=23 -> lower=-1.5707963267948966 upper=3.141592653589793 effort=60 velocity=20
- joint RR_calf_joint: limit lower=-2.7 upper=-0.4 effort=320 velocity=14 -> lower=-2.775 upper=-0.855 effort=60 velocity=20
- joint RR_foot_joint: limit lower=-1000000.0 upper=1000000.0 effort=320 velocity=14 -> lower=-1000000.0 upper=1000000.0 effort=20 velocity=25; origin xyz=0 -0.05 -0.25 rpy=0 0 0 -> xyz=0 -0.08295 -0.25 rpy=0 0 0
- joint RR_hip_joint: limit lower=-0.87 upper=0.87 effort=200 velocity=23 -> lower=-0.7853981633974483 upper=0.7853981633974483 effort=60 velocity=20; origin xyz=-0.1875 -0.075 0 rpy=0 0 0 -> xyz=-0.1875 -0.0725 0 rpy=0 0 0
- joint RR_thigh_joint: limit lower=-1.25 upper=1.25 effort=200 velocity=23 -> lower=-1.5707963267948966 upper=3.141592653589793 effort=60 velocity=20
- joint imu_joint: child imu_link -> imu

Commit message: Enhance terrain, URDF, and logging for improved stability and motion quality

File: resources/wl4/urdf/robot.urdf (robot description, URDF)
Before this commit: robot wl4_description, 19 links, 18 joints
Links:
- link FL_hip: geometry collision cylinder length=0.05 radius=0.05; visual cylinder length=0.05 radius=0.05
- link FR_hip: geometry collision cylinder length=0.05 radius=0.05; visual cylinder length=0.05 radius=0.05
- link RL_hip: geometry collision cylinder length=0.05 radius=0.05; visual cylinder length=0.05 radius=0.05
- link RR_hip: geometry collision cylinder length=0.05 radius=0.05; visual cylinder length=0.05 radius=0.05
Joints:
- joint FL_foot_joint: limit lower=-1000000.0 upper=1000000.0 effort=20 velocity=25 -> lower=-1000000.0 upper=1000000.0 effort=12 velocity=12.5
- joint FR_foot_joint: limit lower=-1000000.0 upper=1000000.0 effort=20 velocity=25 -> lower=-1000000.0 upper=1000000.0 effort=12 velocity=12.5
- joint RL_foot_joint: limit lower=-1000000.0 upper=1000000.0 effort=20 velocity=25 -> lower=-1000000.0 upper=1000000.0 effort=12 velocity=12.5
- joint RR_foot_joint: limit lower=-1000000.0 upper=1000000.0 effort=20 velocity=25 -> lower=-1000000.0 upper=1000000.0 effort=12 velocity=12.5

Commit message: add leg mirror rewards, and modified urdf and onnx output, and changed
Signed-off-by: liu kexin <liukexin@directdrivetech.com>

File: resources/wl4/urdf/robot.urdf (robot description, URDF)
Before this commit: robot wl4_description, 19 links, 18 joints
Links:
- link trunk: mass 8.1 -> 16.2

Commit message: file name change

File: resources/wl4/urdf/robot.urdf (robot description, URDF)
Before this commit: robot wl4_description, 19 links, 18 joints
Links:
- link trunk: geometry collision box size=0.1 0.2 0.3; collision box size=0.1 0.2 0.3
