Commit message: climb 65cm with 4000pt

File: resources/wl4ver2/urdf/robot.urdf (robot description, URDF)
Before this commit: robot wl4v2_description, 17 links, 16 joints
Links:
- link base_link: geometry collision box size=0.049 0.15 0.05; collision box size=0.049 0.15 0.05

Commit message: add wl4v3 robot

File: resources/wl4ver2/urdf/robot.urdf (robot description, URDF)
Before this commit: robot wl4v2_description, 17 links, 16 joints
Joints:
- joint FL_calf_joint: limit lower=-2.775 upper=-0.855 effort=60 velocity=20 -> lower=-2.775 upper=-0.855 effort=80 velocity=20
- joint FL_hip_joint: limit lower=-0.7853981633974483 upper=0.7853981633974483 effort=60 velocity=20 -> lower=-0.7853981633974483 upper=0.7853981633974483 effort=80 velocity=20
- joint FL_thigh_joint: limit lower=-1.5707963267948966 upper=3.141592653589793 effort=60 velocity=20 -> lower=-1.5707963267948966 upper=3.141592653589793 effort=80 velocity=20
- joint FR_calf_joint: limit lower=-2.775 upper=-0.855 effort=60 velocity=20 -> lower=-2.775 upper=-0.855 effort=80 velocity=20
- joint FR_hip_joint: limit lower=-0.7853981633974483 upper=0.7853981633974483 effort=60 velocity=20 -> lower=-0.7853981633974483 upper=0.7853981633974483 effort=80 velocity=20
- joint FR_thigh_joint: limit lower=-1.5707963267948966 upper=3.141592653589793 effort=60 velocity=20 -> lower=-1.5707963267948966 upper=3.141592653589793 effort=80 velocity=20
- joint RL_calf_joint: limit lower=-2.775 upper=-0.855 effort=60 velocity=20 -> lower=-2.775 upper=-0.855 effort=80 velocity=20
- joint RL_hip_joint: limit lower=-0.7853981633974483 upper=0.7853981633974483 effort=60 velocity=20 -> lower=-0.7853981633974483 upper=0.7853981633974483 effort=80 velocity=20
- joint RL_thigh_joint: limit lower=-1.5707963267948966 upper=3.141592653589793 effort=60 velocity=20 -> lower=-1.5707963267948966 upper=3.141592653589793 effort=80 velocity=20
- joint RR_calf_joint: limit lower=-2.775 upper=-0.855 effort=60 velocity=20 -> lower=-2.775 upper=-0.855 effort=80 velocity=20
- joint RR_hip_joint: limit lower=-0.7853981633974483 upper=0.7853981633974483 effort=60 velocity=20 -> lower=-0.7853981633974483 upper=0.7853981633974483 effort=80 velocity=20
- joint RR_thigh_joint: limit lower=-1.5707963267948966 upper=3.141592653589793 effort=60 velocity=20 -> lower=-1.5707963267948966 upper=3.141592653589793 effort=80 velocity=20
