Commit message: refactor: inherit from legged robot

File: resources/go2w/urdf/robot.urdf (robot description, URDF)
Before this commit: robot go2w_description, 33 links, 32 joints
Links:
- link FL_calf: geometry collision cylinder length=0.12 radius=0.012; visual mesh filename=../dae/calf.stl
- link FL_foot: geometry collision cylinder length=0.045 radius=0.086; visual mesh filename=../dae/left_wheel.dae
- link FL_hip: geometry collision cylinder length=0.04 radius=0.046; visual mesh filename=../dae/hip.dae
- link FL_thigh: geometry collision box size=0.11 0.0245 0.034; visual mesh filename=../dae/thigh.dae
- link FR_calf: geometry collision cylinder length=0.12 radius=0.013; visual mesh filename=../dae/calf_mirror.stl
- link FR_foot: geometry collision cylinder length=0.045 radius=0.086; visual mesh filename=../dae/right_wheel.dae
- link FR_hip: geometry collision cylinder length=0.04 radius=0.046; visual mesh filename=../dae/hip.dae
- link FR_thigh: geometry collision box size=0.11 0.0245 0.034; visual mesh filename=../dae/thigh_mirror.dae
- link RL_calf: geometry collision cylinder length=0.12 radius=0.013; visual mesh filename=../dae/calf.stl
- link RL_foot: geometry collision cylinder length=0.045 radius=0.086; visual mesh filename=../dae/left_wheel.dae
- link RL_hip: geometry collision cylinder length=0.04 radius=0.046; visual mesh filename=../dae/hip.dae
- link RL_thigh: geometry collision box size=0.11 0.0245 0.034; visual mesh filename=../dae/thigh.dae
- link RR_calf: geometry collision cylinder length=0.12 radius=0.013; visual mesh filename=../dae/calf_mirror.stl
- link RR_foot: geometry collision cylinder length=0.045 radius=0.086; visual mesh filename=../dae/right_wheel.dae
- link RR_hip: geometry collision cylinder length=0.04 radius=0.046; visual mesh filename=../dae/hip.dae
- link RR_thigh: geometry collision box size=0.11 0.0245 0.034; visual mesh filename=../dae/thigh_mirror.dae
- link base: geometry collision box size=0.3762 0.0935 0.114; visual mesh filename=../dae/base.dae
