Commit message: fix: wl4v3 climb finish , add hopturn and crazy

File: resources/wl4v2/urdf/robot.urdf (robot description, URDF)
Before this commit: robot wl4v2_description, 17 links, 16 joints
Links:
- link base_link: geometry collision box size=0.75 0.15 0.21; collision cylinder length=0.097 radius=0.02
Joints:
- joint FL_calf_joint: limit lower=-2.775 upper=-0.855 effort=80 velocity=20 -> lower=-2.775 upper=-0.855 effort=100 velocity=20
- joint FL_foot_joint: limit lower=-1000000.0 upper=1000000.0 effort=12 velocity=12.5 -> lower=-1000000.0 upper=1000000.0 effort=20 velocity=12.5
- joint FL_hip_joint: limit lower=-0.7853981633974483 upper=0.7853981633974483 effort=80 velocity=20 -> lower=-0.7853981633974483 upper=0.7853981633974483 effort=100 velocity=20
- joint FL_thigh_joint: limit lower=-1.5707963267948966 upper=3.141592653589793 effort=80 velocity=20 -> lower=-1.5707963267948966 upper=3.141592653589793 effort=100 velocity=20
- joint FR_calf_joint: limit lower=-2.775 upper=-0.855 effort=80 velocity=20 -> lower=-2.775 upper=-0.855 effort=100 velocity=20
- joint FR_foot_joint: limit lower=-1000000.0 upper=1000000.0 effort=12 velocity=12.5 -> lower=-1000000.0 upper=1000000.0 effort=20 velocity=12.5
- joint FR_hip_joint: limit lower=-0.7853981633974483 upper=0.7853981633974483 effort=80 velocity=20 -> lower=-0.7853981633974483 upper=0.7853981633974483 effort=100 velocity=20
- joint FR_thigh_joint: limit lower=-1.5707963267948966 upper=3.141592653589793 effort=80 velocity=20 -> lower=-1.5707963267948966 upper=3.141592653589793 effort=100 velocity=20
- joint RL_calf_joint: limit lower=-2.775 upper=-0.855 effort=80 velocity=20 -> lower=-2.775 upper=-0.855 effort=100 velocity=20
- joint RL_foot_joint: limit lower=-1000000.0 upper=1000000.0 effort=12 velocity=12.5 -> lower=-1000000.0 upper=1000000.0 effort=20 velocity=12.5
- joint RL_hip_joint: limit lower=-0.7853981633974483 upper=0.7853981633974483 effort=80 velocity=20 -> lower=-0.7853981633974483 upper=0.7853981633974483 effort=100 velocity=20
- joint RL_thigh_joint: limit lower=-1.5707963267948966 upper=3.141592653589793 effort=80 velocity=20 -> lower=-1.5707963267948966 upper=3.141592653589793 effort=100 velocity=20
- joint RR_calf_joint: limit lower=-2.775 upper=-0.855 effort=80 velocity=20 -> lower=-2.775 upper=-0.855 effort=100 velocity=20
- joint RR_foot_joint: limit lower=-1000000.0 upper=1000000.0 effort=12 velocity=12.5 -> lower=-1000000.0 upper=1000000.0 effort=20 velocity=12.5
- joint RR_hip_joint: limit lower=-0.7853981633974483 upper=0.7853981633974483 effort=80 velocity=20 -> lower=-0.7853981633974483 upper=0.7853981633974483 effort=100 velocity=20
- joint RR_thigh_joint: limit lower=-1.5707963267948966 upper=3.141592653589793 effort=80 velocity=20 -> lower=-1.5707963267948966 upper=3.141592653589793 effort=100 velocity=20

File: resources/wl4v3/urdf/robot.urdf (robot description, URDF)
Before this commit: robot wl4v3_description, 19 links, 18 joints
Joints:
- joint FL_calf_joint: limit lower=-2.775 upper=-0.855 effort=80 velocity=20 -> lower=-2.775 upper=-0.855 effort=80 velocity=15
- joint FL_foot_joint: limit lower=-1000000.0 upper=1000000.0 effort=12 velocity=12.5 -> lower=-1000000.0 upper=1000000.0 effort=20 velocity=12.5
- joint FL_hip_joint: limit lower=-0.7853981633974483 upper=0.7853981633974483 effort=80 velocity=20 -> lower=-0.7853981633974483 upper=0.7853981633974483 effort=80 velocity=15
- joint FL_thigh_joint: limit lower=-1.5707963267948966 upper=3.141592653589793 effort=80 velocity=20 -> lower=-1.5707963267948966 upper=3.141592653589793 effort=80 velocity=15
- joint FR_calf_joint: limit lower=-2.775 upper=-0.855 effort=80 velocity=20 -> lower=-2.775 upper=-0.855 effort=80 velocity=15
- joint FR_foot_joint: limit lower=-1000000.0 upper=1000000.0 effort=12 velocity=12.5 -> lower=-1000000.0 upper=1000000.0 effort=20 velocity=12.5
- joint FR_hip_joint: limit lower=-0.7853981633974483 upper=0.7853981633974483 effort=80 velocity=20 -> lower=-0.7853981633974483 upper=0.7853981633974483 effort=80 velocity=15
- joint FR_thigh_joint: limit lower=-1.5707963267948966 upper=3.141592653589793 effort=80 velocity=20 -> lower=-1.5707963267948966 upper=3.141592653589793 effort=80 velocity=15
- joint RL_calf_joint: limit lower=-2.775 upper=-0.855 effort=80 velocity=20 -> lower=-2.775 upper=-0.855 effort=80 velocity=15
- joint RL_foot_joint: limit lower=-1000000.0 upper=1000000.0 effort=12 velocity=12.5 -> lower=-1000000.0 upper=1000000.0 effort=20 velocity=12.5
- joint RL_hip_joint: limit lower=-0.7853981633974483 upper=0.7853981633974483 effort=80 velocity=20 -> lower=-0.7853981633974483 upper=0.7853981633974483 effort=80 velocity=15
- joint RL_thigh_joint: limit lower=-1.5707963267948966 upper=3.141592653589793 effort=80 velocity=20 -> lower=-1.5707963267948966 upper=3.141592653589793 effort=80 velocity=15
- joint RR_calf_joint: limit lower=-2.775 upper=-0.855 effort=80 velocity=20 -> lower=-2.775 upper=-0.855 effort=80 velocity=15
- joint RR_foot_joint: limit lower=-1000000.0 upper=1000000.0 effort=12 velocity=12.5 -> lower=-1000000.0 upper=1000000.0 effort=20 velocity=12.5
- joint RR_hip_joint: limit lower=-0.7853981633974483 upper=0.7853981633974483 effort=80 velocity=20 -> lower=-0.7853981633974483 upper=0.7853981633974483 effort=80 velocity=15
- joint RR_thigh_joint: limit lower=-1.5707963267948966 upper=3.141592653589793 effort=80 velocity=20 -> lower=-1.5707963267948966 upper=3.141592653589793 effort=80 velocity=15
