Commit message: fix: init tita config and y1v0 config,  delete useless actor_critic

File: resources/wl4v3/urdf/robot.urdf (robot description, URDF)
Before this commit: robot wl4v3_description, 19 links, 18 joints
Joints:
- joint FL_foot_joint: limit lower=-1000000.0 upper=1000000.0 effort=20 velocity=12.5 -> lower=-1000000.0 upper=1000000.0 effort=20 velocity=25
- joint FR_foot_joint: limit lower=-1000000.0 upper=1000000.0 effort=20 velocity=12.5 -> lower=-1000000.0 upper=1000000.0 effort=20 velocity=25
- joint RL_foot_joint: limit lower=-1000000.0 upper=1000000.0 effort=20 velocity=12.5 -> lower=-1000000.0 upper=1000000.0 effort=20 velocity=25
- joint RR_foot_joint: limit lower=-1000000.0 upper=1000000.0 effort=20 velocity=12.5 -> lower=-1000000.0 upper=1000000.0 effort=20 velocity=25
